File: aquanode-kicad.kicad_sch (KiCad schematic)
At the start: 24 parts, among them J1 Conn_01x04, J2 Conn_01x03, J3 Conn_01x02, Q1 BC817, U1 XIAO-ESP32-C6, U2 AMS1117-3.3, U3 AMS1117-5.0

Commit message: asignar huellas
Parts:
- removed D1: LED, symbol Device:LED
- added D1: 1N4148, Diode_THT:D_DO-35_SOD27_P7.62mm_Horizontal, symbol Diode:1N4148
- added D2: LED, symbol Device:LED
- added K1: RM50-xx21, Relay_THT:Relay_SPST_Finder_32.21-x300, symbol Relay:RM50-xx21
- added R2: 1k, symbol Device:R
- renumbered C11 to C1, C7 to C10, C8 to C11, C9 to C2, C10 to C3, C1 to C4, C3 to C5, C5 to C6, C4 to C7, C2 to C8, C6 to C9, U2 to U1, U3 to U2, U1 to U3
Connections:
- net +12V: now also D1.1 (K), K1.11, K1.A2, R2.1
- net +3V3: now also U1.2 (VO); no longer U1.1 (GND)
- net +5V: now also U2.2 (VO); no longer U2.1 (GND)
- net GND: now also Q1.2 (E), U1.1 (GND), U2.1 (GND); no longer U1.2 (VO), U2.2 (VO)
- net r: now reaches Q1.3 (C)
- net r: now also D1.2 (A), D2.1 (K), K1.A1
- net rOut: no longer names the net of J3.2 (Pin_2)
- net rOut: now also K1.14
- new net: D2.2 (A), R2.2
Other:
- moved on the sheet: J3, Q1, R1

Commit message: huellas
Parts:
- C1: footprint (none) -> Capacitor_THT:CP_Radial_D8.0mm_P5.00mm
- C2: footprint (none) -> Capacitor_SMD:CP_Elec_3x5.3
- C7: footprint (none) -> Capacitor_THT:CP_Radial_D8.0mm_P3.80mm
Connections:
- no-connect marks 0 -> 10
Changed lines of the file:
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@@
 		(color 0 0 0 0)
 	)
+	(no_connect
+		(at 227.33 92.71)
+	)
+	(no_connect
+		(at 177.8 85.09)
+	)
+	(no_connect
+		(at 227.33 96.52)
+	)
+	(no_connect
+		(at 227.33 88.9)
+	)
+	(no_connect
+		(at 177.8 88.9)
+	)
+	(no_connect
+		(at 227.33 100.33)
+	)
+	(no_connect
+		(at 177.8 92.71)
+	)
+	(no_connect
+		(at 177.8 100.33)
+	)
+	(no_connect
+		(at 227.33 77.47)
+	)
+	(no_connect
+		(at 177.8 96.52)
+	)
 	(wire
 		(pts
@@
 			)
 		)
-		(property "Footprint" ""
+		(property "Footprint" "Capacitor_SMD:CP_Elec_3x5.3"
 			(at 188.9252 144.78 0)
 			(effects
@@
 			)
 		)
-		(property "Footprint" ""
+		(property "Footprint" "Capacitor_THT:CP_Radial_D8.0mm_P5.00mm"
 			(at 182.5752 144.78 0)
 			(effects
@@
 			)
 		)
-		(property "Footprint" ""
+		(property "Footprint" "Capacitor_THT:CP_Radial_D8.0mm_P3.80mm"
 			(at 229.5652 144.78 0)
 			(effects

Commit message: ??
Parts:
- removed C1: 220u, Capacitor_THT:CP_Radial_D8.0mm_P5.00mm, symbol Device:C_Polarized
- removed C10, C6: 22u, symbol Device:C_Polarized
- removed C11: 22uF, symbol Device:C
- removed C2: 10uF, Capacitor_SMD:CP_Elec_3x5.3, symbol Device:C
- removed C3, C5, C9: 0.1u, symbol Device:C
- removed C7: 22uF, Capacitor_THT:CP_Radial_D8.0mm_P3.80mm, symbol Device:C
- removed U1: AMS1117-3.3, Package_TO_SOT_SMD:SOT-223-3_TabPin2, symbol Regulator_Linear:AMS1117-3.3
- removed U2: AMS1117-5.0, Package_TO_SOT_SMD:SOT-223-3_TabPin2, symbol Regulator_Linear:AMS1117-5.0
- added C12, C15, C20: 10u, symbol Device:C
- added C13, C18: 22uF, symbol Device:C
- added C14: 220u, Capacitor_THT:CP_Radial_D8.0mm_P3.80mm, symbol Device:C_Polarized
- added C16: 0.1u, Capacitor_SMD:C_0603_1608Metric_Pad1.08x0.95mm_HandSolder, symbol Device:C
- added C17, C19: 22uF, Capacitor_Tantalum_SMD:CP_EIA-2012-15_AVX-P_HandSolder, symbol Device:C
- added L1: 47uH, Inductor_SMD:L_1812_4532Metric, symbol Device:L
- added U1, U2: K78XX, JS_Devices:K78XX, symbol JS_Devices:K78XX
Connections:
- net +12V: now also C12.1, C14.1, C15.1, C16.1, C20.1, U1.1 (VI), U2.1 (VI)
- net +3V3: now also C17.1, L1.2
- net +5V: now also C18.1, C19.1, U2.3 (VO)
- net GND: now also C12.2, C13.2, C14.2, C15.2, C16.2, C17.2, C18.2, C19.2, C20.2, U1.2 (GND), U2.2 (GND)
- new net: C13.1, L1.1, U1.3 (VO)
Other:
- moved on the sheet: C4, J1
